File: osu keyboard.kicad_sch (KiCad schematic)
At the start: 20 parts, among them SW1 SW_Push, Y1 16MHz

Commit message: Schematics
Parts:
- removed D? (x2): SOD-123, symbol Device:D_Small
- removed USB?: Molex-0548190589, symbol random-keyboard-parts:Molex-0548190589
- added C8, C9: 0.1uF, Capacitor_SMD:C_0805_2012Metric, symbol Device:C_Small
- added D1, D4: WS2812B, LED_SMD:LED_WS2812B_PLCC4_5.0x5.0mm_P3.2mm, symbol LED:WS2812B
- added R5, R6: 5.1k, Resistor_SMD:R_0805_2012Metric, symbol Device:R_Small
- added U2: PRTR5V0U2X, random-keyboard-parts:SOT143B, symbol random-keyboard-parts:PRTR5V0U2X
- added USB1: HRO-TYPE-C-31-M-12, Type-C:HRO-TYPE-C-31-M-12, symbol Type-C:HRO-TYPE-C-31-M-12
- C1, C2, C3, C4, C5, C6, C7: footprint (none) -> Capacitor_SMD:C_0805_2012Metric
- F1: footprint (none) -> Fuse:Fuse_1206_3216Metric
- MX0, MX1: renamed from MX?; footprint (none) -> MX_Alps_Hybrid:MX-1U
- R1, R3, R4: footprint (none) -> Resistor_SMD:R_0805_2012Metric
- R2: value R_Small -> 22; footprint (none) -> Resistor_SMD:R_0805_2012Metric
- SW1: footprint (none) -> random-keyboard-parts:SKQG-1155865
- Y1: footprint (none) -> Crystal:Crystal_SMD_3225-4Pin_3.2x2.5mm
- gave numbers to parts that had none: 1
Connections:
- net +5V: now also F1.1, MX0.3 (LED), MX1.3 (LED), C8.2, C9.2, D1.1 (VDD), D4.1 (VDD); no longer F1.2
- net D+: now also U2.2 (IO1), USB1.6 (DP1), USB1.8 (DP2)
- net D-: now also U2.3 (IO2), USB1.5 (DN2), USB1.7 (DN1)
- net GND: now also MX0.2 (ROW), MX0.4 (LEDGND), MX1.2 (ROW), MX1.4 (LEDGND), C8.1, C9.1, D1.3 (VSS), D4.3 (VSS), R5.2, R6.2, U2.1 (GND), USB1.1 (GND), USB1.12 (GND), USB1.13 (SHIELD)
- net VCC: now also F1.2, U2.4 (VCC), USB1.11 (VBUS), USB1.2 (VBUS); no longer F1.1
- net XTAL1: now reaches C1.2, U1.17 (XTAL1), Y1.1
- net UNDERGLOWLED: now reaches U1.11 (PB3)
- net UNDERGLOWLED: now also D4.4 (DIN)
- net XTAL2: now reaches C2.2, U1.16 (XTAL2), Y1.3
- net ROW0: no longer names the net of U1.27 (PD7)
- new net: R5.1, USB1.10 (CC2)
- new net: R6.1, USB1.4 (CC1)
- new net: D1.4 (DIN), D4.2 (DOUT)
Other:
- moved on the sheet: C1, C2, C3, C4, C5, C6, C7, MX0, MX1, R1, R2, R3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

Commit message: pcb setup arranged
Parts:
- C3: value C_Small -> 1uF
Changed lines of the file:
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@@
       (effects (font (size 1.27 1.27)) (justify left))
     )
-    (property "Value" "C_Small" (id 1) (at 41.91 76.2062 0)
+    (property "Value" "1uF" (id 1) (at 41.91 76.2062 0)
       (effects (font (size 1.27 1.27)) (justify left))
     )
@@
     )
     (path "/332dd123-7a8f-4d5b-afc7-271f8484b7c3"
-      (reference "C3") (unit 1) (value "C_Small") (footprint "Capacitor_SMD:C_0805_2012Metric")
+      (reference "C3") (unit 1) (value "1uF") (footprint "Capacitor_SMD:C_0805_2012Metric")
     )
     (path "/f24c34fa-3957-4d04-998c-9ce6fa0302c1"
